File: gitkicadtutorial/gitkicadtutorial.kicad_pcb (KiCad board)
At the start: 2 copper layers, 7 parts, among them CN1 CON_PIN_HEADER_1X6_2.54_180_1, U1 LM1117-3.3, U2 ESP32-S3-WROOM-1-N8

Commit message: esquematico finalizado
Parts:
- added C1: CAP_1U_50V_0805_X7R, minha_lib:CAP_0805, F.Cu at (165.1, 101.6)
- added C2: CAP_100N_50V_0805_X7R, minha_lib:CAP_0805, F.Cu at (165.1, 104.4)
- added C3: CAP_1U_50V_0805_X7R, minha_lib:CAP_0805, F.Cu at (176.5, 98.9)
- added CN2: CON_PIN_HEADER_1X6_2.54_180_1, minha_lib:pin_header_male_6_2.54_pth, F.Cu at (160.2, 95.6)
- added LD1: LED_VERDE_0805_L171L-GC-TR, minha_lib:LED_0805, F.Cu at (171.8, 98.8)
- added LD2: LED_VERDE_0805_L171L-GC-TR, minha_lib:LED_0805, F.Cu at (161.2, 98.8)
- added LD3: LED_VERDE_0805_L171L-GC-TR, minha_lib:LED_0805, F.Cu at (166.6, 98.8)
- added R5: R_0805_1K_1%_1/8W, minha_lib:RES_0805, F.Cu at (177.0, 95.2)
- added R6: R_0805_1K_1%_1/8W, minha_lib:RES_0805, F.Cu at (160.6, 104.4)
- added R7: R_0805_1K_1%_1/8W, minha_lib:RES_0805, F.Cu at (160.6, 101.6)
Connections:
- CN1 pad 4: /TX -> unconnected-(CN1-Pad4)
- CN1 pad 5: Net-(CN1-Pad5) -> unconnected-(CN1-Pad5)
- CN1 pad 6: Net-(CN1-Pad6) -> unconnected-(CN1-Pad6)
- R1 pad 1: Net-(CN1-Pad6) -> unconnected-(R1-Pad1)
- R2 pad 2: Net-(CN1-Pad6) -> unconnected-(R2-Pad2)
- R3 pad 2: Net-(R3-Pad2) -> unconnected-(R3-Pad2)
- R4 pad 2: Net-(R4-Pad2) -> unconnected-(R4-Pad2)
- U2 pad 12: unconnected-(U2-Pad12) -> Net-(U2-Pad12)
- U2 pad 13: unconnected-(U2-Pad13) -> Net-(U2-Pad13)
- U2 pad 14: unconnected-(U2-Pad14) -> Net-(U2-Pad14)
- U2 pad 16: Net-(R3-Pad2) -> unconnected-(U2-Pad16)
- U2 pad 26: Net-(R4-Pad2) -> unconnected-(U2-Pad26)
- U2 pad 27: /BOOT -> unconnected-(U2-Pad27)
- U2 pad 3: Net-(CN1-Pad5) -> unconnected-(U2-Pad3)
- U2 pad 36: /RX -> unconnected-(U2-Pad36)
- U2 pad 37: /TX -> unconnected-(U2-Pad37)
- U2 pad 40: GND -> unconnected-(U2-Pad40)
- U2 pad 41: GND -> unconnected-(U2-Pad41)

Commit message: esquematico revisado
Parts:
- CN1, CN2: value CON_PIN_HEADER_1X6_2.54_180_1 -> CON_PIN_HEADER_1X6_2.54_180
- U2: value ESP32-S3-WROOM-1-N8 -> UC_ESP32-S3-WROOM-1-N8
- moved CN2 52.0 mm to (109.0, 104.6), turned to 90 degrees
- moved LD1 33.0 mm to (138.9, 100.7)
- moved C3 31.6 mm to (151.6, 79.4)
- moved CN1 31.6 mm to (109.0, 75.7), turned to -90 degrees
- moved R2 31.3 mm to (117.0, 81.0), turned to 180 degrees
- moved C1 29.2 mm to (159.0, 73.0)
- moved R7 28.9 mm to (165.1, 73.0)
- moved R6 28.6 mm to (160.6, 75.8)
- moved C2 28.3 mm to (142.6, 87.3)
- moved LD3 26.4 mm to (152.2, 76.7)
- moved R3 24.9 mm to (156.1, 79.4)
- moved R5 24.6 mm to (156.1, 82.2)
- moved LD2 23.0 mm to (143.2, 84.5)
- moved R4 12.7 mm to (160.6, 78.6)
- moved R1 10.4 mm to (151.6, 82.2)
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Connections:
- CN1 pad 4: unconnected-(CN1-Pad4) -> /TX
- CN1 pad 5: unconnected-(CN1-Pad5) -> Net-(U2-Pad3)
- CN1 pad 6: unconnected-(CN1-Pad6) -> Net-(R1-Pad1)
- CN2 pad 4: unconnected-(CN2-Pad4) -> Net-(U2-Pad11)
- CN2 pad 5: unconnected-(CN2-Pad5) -> Net-(U2-Pad10)
- CN2 pad 6: unconnected-(CN2-Pad6) -> Net-(U2-Pad9)
- LD1 pad 2: unconnected-(LD1-Pad2) -> Net-(LD1-Pad2)
- LD2 pad 2: unconnected-(LD2-Pad2) -> Net-(LD2-Pad2)
- LD3 pad 2: unconnected-(LD3-Pad2) -> Net-(LD3-Pad2)
- R1 pad 1: unconnected-(R1-Pad1) -> Net-(R1-Pad1)
- R2 pad 2: unconnected-(R2-Pad2) -> Net-(R1-Pad1)
- R3 pad 2: unconnected-(R3-Pad2) -> Net-(R3-Pad2)
- R4 pad 2: unconnected-(R4-Pad2) -> Net-(R4-Pad2)
- R5 pad 1: unconnected-(R5-Pad1) -> Net-(R5-Pad1)
- R5 pad 2: unconnected-(R5-Pad2) -> Net-(LD1-Pad2)
- R6 pad 1: unconnected-(R6-Pad1) -> Net-(R6-Pad1)
- R6 pad 2: unconnected-(R6-Pad2) -> Net-(LD2-Pad2)
- R7 pad 1: unconnected-(R7-Pad1) -> Net-(R7-Pad1)
- R7 pad 2: unconnected-(R7-Pad2) -> Net-(LD3-Pad2)
- U2 pad 10: unconnected-(U2-Pad10) -> Net-(U2-Pad10)
- U2 pad 11: unconnected-(U2-Pad11) -> Net-(U2-Pad11)
- U2 pad 16: unconnected-(U2-Pad16) -> Net-(R3-Pad2)
- U2 pad 26: unconnected-(U2-Pad26) -> Net-(R4-Pad2)
- U2 pad 27: unconnected-(U2-Pad27) -> /BOOT
- U2 pad 3: unconnected-(U2-Pad3) -> Net-(U2-Pad3)
- U2 pad 32: unconnected-(U2-Pad32) -> Net-(R7-Pad1)
- U2 pad 33: unconnected-(U2-Pad33) -> Net-(R6-Pad1)
- U2 pad 34: unconnected-(U2-Pad34) -> Net-(R5-Pad1)
- U2 pad 36: unconnected-(U2-Pad36) -> /RX
- U2 pad 37: unconnected-(U2-Pad37) -> /TX
- U2 pad 40: unconnected-(U2-Pad40) -> GND
- U2 pad 41: unconnected-(U2-Pad41) -> GND
- U2 pad 9: unconnected-(U2-Pad9) -> Net-(U2-Pad9)
