File: gitkicadtutorial/gitkicadtutorial.kicad_sch (KiCad schematic)
At the start: 10 parts, among them CN1 CON_PIN_HEADER_1X6_2.54_180_1, U1 LM1117-3.3, U2 ESP32-S3-WROOM-1-N8

Commit message: esquematico finalizado
Parts:
- added CN2: (no value), symbol minha_lib_:CON_PIN_HEADER_1X6_2.54_180_1
- added LD1, LD2, LD3: (no value), symbol minha_lib_:LED_VERDE_0805_L171L-GC-TR
- added R5, R6, R7: (no value), symbol minha_lib_:R_0805_1K_1%_1/8W
Connections:
- net GND: now also LD1.1 (CATHODE), LD2.1 (CATHODE), LD3.1 (CATHODE)
- net at U2.10 (IO17): now also CN2.5
- net at U2.11 (IO18): now also CN2.4
- net at U2.12 (IO8): now also CN2.3
- net at U2.13 (IO19): now also CN2.2
- net at U2.14 (IO20): now also CN2.1
- net at U2.32 (IO39): now also R7.1 (CATHODE)
- net at U2.33 (IO40): now also R6.1 (CATHODE)
- net at U2.34 (IO41): now also R5.1 (CATHODE)
- net at U2.9 (IO16): now also CN2.6
- new net: LD2.2 (ANODE), R6.2 (ANODE)
- new net: LD1.2 (ANODE), R5.2 (ANODE)
- new net: LD3.2 (ANODE), R7.2 (ANODE)
- no-connect marks 0 -> 22

Commit message: esquematico revisado
Parts:
- removed CN1: CON_PIN_HEADER_1X6_2.54_180_1, minha_lib:pin_header_male_6_2.54_pth, symbol minha_lib_:CON_PIN_HEADER_1X6_2.54_180_1
- removed CN2: (no value), symbol minha_lib_:CON_PIN_HEADER_1X6_2.54_180_1
- removed U2: ESP32-S3-WROOM-1-N8, minha_lib:ESP32-S3-WROOM-1, symbol minha_lib_:ESP32-S3-WROOM-1-N8
- added CN1, CN2: CON_PIN_HEADER_1X6_2.54_180, minha_lib:pin_header_male_6_2.54_pth, symbol minha_lib_:CON_PIN_HEADER_1X6_2.54_180
- added U2: UC_ESP32-S3-WROOM-1-N8, minha_lib:ESP32-S3-WROOM-1, symbol minha_lib_:UC_ESP32-S3-WROOM-1-N8
- C1, C2, C3: footprint (none) -> minha_lib:CAP_0805
- LD1, LD2, LD3: value (none) -> LED_VERDE_0805_L171L-GC-TR; footprint (none) -> minha_lib:LED_0805
- R5, R6, R7: value (none) -> R_0805_1K_1%_1/8W; footprint (none) -> minha_lib:RES_0805
Connections:
- net +3V3: now also U2.2 (3V3)
- net BOOT: now also CN1.2, U2.27 (IO0)
- net GND: now also CN1.1, U2.1 (GND), U2.40 (GND), U2.41 (GND)
- net RX: now also CN1.3, U2.36 (RXD0)
- net TX: now also CN1.4, U2.37 (TXD0)
- net at R5.1 (CATHODE): now also U2.34 (IO41)
- net at R3.2 (ANODE): now also U2.16 (IO46)
- net at R4.2 (ANODE): now also U2.26 (IO45)
- net at R7.1 (CATHODE): now also U2.32 (IO39)
- net at R6.1 (CATHODE): now also U2.33 (IO40)
- net at R1.1 (CATHODE), R2.2 (ANODE): now also CN1.6
- new net: CN2.1, U2.14 (IO20)
- new net: CN2.2, U2.13 (IO19)
- new net: CN2.3, U2.12 (IO8)
- new net: CN2.4, U2.11 (IO18)
- new net: CN2.5, U2.10 (IO17)
- new net: CN2.6, U2.9 (IO16)
- new net: CN1.5, U2.3 (EN)
Other:
- title: (none) -> GIT KiCad Tutorial
